Commit message: Add files via upload

File: my_edu_rover_description/urdf/wheel/wheel.gazebo.xacro (robot description, xacro)
@@ -1,9 +1,10 @@
 <?xml version="1.0"?>
 <robot xmlns:xacro="http://ros.org/wiki/xacro">
-  <xacro:macro name="wheel_gazebo_v0" params="prefix">
-    <gazebo reference="${prefix}_wheel_link">
+  <xacro:macro name="wheel_gazebo" params="number">
+    <gazebo reference="wheel_${number}_link">
       <selfCollide>false</selfCollide>
       <mu1 value="1.2" />
       <mu2 value="1.2" />
+      <material>Gazebo/Black</material>
     </gazebo>
   </xacro:macro>

File: my_edu_rover_description/urdf/wheel/wheel.transmission.xacro (robot description, xacro)
@@ -1,11 +1,11 @@
 <?xml version="1.0"?>
 <robot xmlns:xacro="http://ros.org/wiki/xacro">
-  <xacro:macro name="wheel_trans_v0" params="prefix">
-    <transmission name="${prefix}_wheel_trans">
+  <xacro:macro name="wheel_transmission" params="number">
+    <transmission name="wheel_${number}_transmission">
       <type>transmission_interface/SimpleTransmission</type>
-      <joint name="${prefix}_wheel_joint">
+      <joint name="wheel_${number}_joint">
 	<hardwareInterface>hardware_interface/VelocityJointInterface</hardwareInterface>
       </joint>
-	<actuator name="${prefix}_wheel_motor">
+	<actuator name="wheel_${number}_motor">
 	  <hardwareInterface>hardware_interface/VelocityJointInterface</hardwareInterface>
 	  <mechanicalReduction>1</mechanicalReduction>

File: my_edu_rover_description/urdf/wheel/wheel.urdf.xacro (robot description, xacro)
@@ -1,29 +1,29 @@
 <?xml version="1.0"?>
 <robot xmlns:xacro="http://ros.org/wiki/xacro">
-  <xacro:include filename="$(find fourth_robot_description)/urdf/wheel/wheel.transmission.xacro"/>
-  <xacro:include filename="$(find fourth_robot_description)/urdf/wheel/wheel.gazebo.xacro"/>
-  <xacro:macro name="wheel_v0" params="prefix parent *joint_origin *joint_axis">
-	<joint name="${prefix}_wheel_joint" type="continuous">
-	  <xacro:insert_block name="joint_origin"/>
-	  <parent link="${parent}"/>
-	  <child link="${prefix}_wheel_link"/>
+  <xacro:include filename="$(find my_edu_rover_description)/urdf/wheel/wheel.transmission.xacro"/>
+  <xacro:include filename="$(find my_edu_rover_description)/urdf/wheel/wheel.gazebo.xacro"/>
+  <xacro:macro name="wheel" params="number xyz rpy">
+	<joint name="wheel_${number}_joint" type="continuous">
+	  <origin xyz = "${xyz}" rpy = "${rpy}"/>
+	  <parent link="knuckle_${number}_link"/>
+	  <child link="wheel_${number}_link"/>
          <limit effort="1.5" velocity="20"/>
-	  <xacro:insert_block name="joint_axis"/>
+	  <axis xyz = "0 1 0"/>
 	</joint>
-	<link name="${prefix}_wheel_link">
+	<link name="wheel_${number}_link">
 	  <visual>
 		<geometry>
-		  <mesh filename="package://fourth_robot_description/meshes/DAE/wheel/wheel_link.dae"/>
+		  <mesh filename="package://my_edu_rover_description/models/wheel.STL"/>
 		</geometry>
 	  </visual>
 	  <collision>
 		<geometry>
-		  <mesh filename="package://fourth_robot_description/meshes/STL/wheel/robot_wheel.stl"/>
+		  <mesh filename="package://my_edu_rover_description/models/wheel.STL"/>
 		</geometry>
 	  </collision>
 	  <inertial>
-		<origin xyz="0.0 -0.007 -0.0"/>
-		<mass value="0.05"/>
-		<inertia ixx="0.00001" ixy="0" ixz="0" iyy="0.000018" iyz="0" izz="0.00001"/>
+        <origin xyz = "0 0 0" rpy = "0 0 0"/>
+        <mass value = "0.038593"/>
+		<inertia ixx = "1.5759e-05" ixy = "0.0" ixz = "0.0" iyy = "1.5759e-05" iyz = "0.0" izz = "3.0874e-05"/>
 	  </inertial>
 	</link>
